File: KiCAD/boards/DevBoard/DevBoard.kicad_sch (KiCad schematic)
At the start: 7 parts, among them J1 Conn_ARM_SWD_TagConnect_TC203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, J2 Conn_01x09, J3 Conn_01x08, J4 Conn_01x08, U1 STM32C092FCP6, U2 SN65HVD232QDRG4Q1, U3 SST25PF020B-80-4C-SAE

Commit message: DevBoard first revision
Parts:
- added C1, C3, C4, C5: 100n, Capacitor_SMD:C_0603_1608Metric, symbol Device:C
- added C2: 10u, Capacitor_SMD:C_0603_1608Metric, symbol Device:C
- added D1: LED, LED_SMD:LED_0603_1608Metric, symbol Device:LED
- added R1: 1k, Resistor_SMD:R_0603_1608Metric, symbol Device:R
Connections:
- net 3V3 is gone; now on net +3V3: J4.1 (Pin_1)
- net +3V3: now also C1.1, C2.1, C3.1, C4.1, C5.1, D1.2 (A)
- net GND: now also C1.2, C2.2, C3.2, C4.2, C5.2, R1.2
- new net: D1.1 (K), R1.1
