File: KiCAD/boards/TC3Controller/TC3Controller.kicad_pcb (KiCad board)
At the start: 2 copper layers, 35 x 37.3 mm, 39 parts, among them J1 Conn_ARM_SWD_TagConnect_TC203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, J2 Screw_Terminal_01x02, J3 Screw_Terminal_01x02, J4 Screw_Terminal_01x02, J5 Conn_01x05, J6 Conn_01x05, U1 STM32C092FCP6, U2 SN65HVD232QDRG4Q1, U3 SST25PF020B-80-4C-SAE, U4 MAX31855KASA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

Commit message: Servo controller board & fixes to TC board
Parts:
- moved C5 0.57 mm to (132.3, 67.6)
Connections:
- J6 pad 1: /RESETB -> +3V3
- J6 pad 2: GND -> /CAN+
- J6 pad 4: /CAN+ -> GND
- J6 pad 5: +3V3 -> /RESETB
Routing:
- net GND: track 157.4 -> 138.2 mm, vias 17 -> 22
- net /RESETB: track 53.6 -> 57.9 mm, vias 1 -> 3
- net /SWO: track 16.2 -> 19.1 mm
- net /CAN+: track 33.7 -> 31.4 mm, vias 1 -> 0
- net +3V3: track 154.3 -> 152.1 mm, vias 4 -> 5
- net /CAN-: track 35.7 -> 34.5 mm
- net /TC2_CS: track 14.8 -> 14.0 mm
Other:
- board text added: "Papyrus System"
- board text removed: "Athena DAQ System"
